File: 4001_4153_LO_V2.sch (EAGLE design)
At the start: 117 parts, among them IC1 74LVC2G17GV,125, IC10 MCP6H01T-E/LT, IC11 TL431AIDBZR, IC2 74LVC2G17GV,125, IC3 74LVC2G17GV,125, IC4 ADF4001BRUZ, IC5 ATTINY45V-10SU, IC6 7805DT, IC7 7809DT, IC8 LD1117AS33TR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

Commit message: various
Parts:
- removed R19: 51R, rcl:R-EU_R0603
- C22: value 100nF -> 100pF; device rcl:C-EUC0805 -> resistor:C-EUC0603
- IC10: value MCP6H01T-E/LT -> TS971ILT; MPN MCP6H01T-E/LT -> TS971ILT; OC_FARNELL 2920751 -> 9755730
- R18: value 18K -> 22R
Connections:
- removed net CLK: IC4.CLK, IC9.CLK
- new net +5V_VCO: L6.2
- net +9V: no longer C22.1, L6.2
- net GND: no longer R19.1
- net N$1: now also C22.1; no longer R19.2
- net SCK: now also IC4.CLK, IC9.CLK
Other:
- moved on the sheet: C22, SJ1
Changed lines of the file:
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@@
 </classes>
 <parts>
-<part name="C22" library="rcl" deviceset="C-EU" device="C0805" value="100nF"/>
 <part name="SUPPLY3" library="supply2" deviceset="DGND" device="" value="AGND"/>
 <part name="AGND39" library="supply1" deviceset="AGND" device=""/>
@@
 <part name="U$5" library="Document" deviceset="DOC_DOCFIELD_CCSA" device=""/>
 <part name="IC9" library="ADF4153BRUZ-RL7" deviceset="ADF4153BRUZ-RL7" device=""/>
-<part name="R19" library="rcl" deviceset="R-EU_" device="R0603" value="51R"/>
 <part name="C36" library="resistor" deviceset="C-EU" device="C0603" value="1uF"/>
 <part name="C37" library="resistor" deviceset="C-EU" device="C0603" value="100nF"/>
@@
 <part name="L6" library="resistor" deviceset="R-EU_" device="R0603" value="100nH"/>
 <part name="L11" library="resistor" deviceset="R-EU_" device="R0603" value="100nH"/>
-<part name="IC10" library="RF" deviceset="MCP6H01" device="" value="MCP6H01T-E/LT ">
-<attribute name="MPN" value="MCP6H01T-E/LT "/>
-<attribute name="OC_FARNELL" value="2920751"/>
+<part name="IC10" library="RF" deviceset="MCP6H01" device="" value="TS971ILT ">
+<attribute name="MPN" value="TS971ILT "/>
+<attribute name="OC_FARNELL" value="9755730"/>
 </part>
 <part name="R25" library="rcl" deviceset="R-EU_" device="R0603" value="10K"/>
@@
 <part name="R23" library="rcl" deviceset="R-EU_" device="R0603" value="5K1"/>
 <part name="R16" library="rcl" deviceset="R-EU_" device="R0603" value="TO TASTE"/>
-<part name="R18" library="rcl" deviceset="R-EU_" device="R0603" value="18K"/>
+<part name="R18" library="rcl" deviceset="R-EU_" device="R0603" value="22R"/>
 <part name="C42" library="resistor" deviceset="C-EU" device="C0603" value="100pF"/>
 <part name="Q1" library="zetex" deviceset="NMOSSOT89" device="" value="PGA105+"/>
@@
 <part name="R32" library="rcl" deviceset="R-EU_" device="R0603" value="10K"/>
 <part name="C4" library="rcl" deviceset="C-EU" device="C0603" value="100nF"/>
+<part name="C22" library="resistor" deviceset="C-EU" device="C0603" value="100pF"/>
 </parts>
 <sheets>
@@
 <instance part="C26" gate="G$1" x="383.54" y="165.1"/>
 <instance part="C27" gate="G$1" x="419.1" y="165.1"/>
-<instance part="C22" gate="G$1" x="462.28" y="198.12"/>
 <instance part="SUPPLY3" gate="G$1" x="464.82" y="182.88"/>
 <instance part="IC7" gate="A1" x="401.32" y="205.74"/>
@@
 <instance part="U$5" gate="CCSA" x="515.62" y="0"/>
 <instance part="IC9" gate="G$1" x="190.5" y="81.28" rot="R180"/>
-<instance part="R19" gate="G$1" x="203.2" y="91.44" rot="R180"/>
 <instance part="AGND39" gate="VR1" x="175.26" y="160.02"/>
 <instance part="C24" gate="G$1" x="147.32" y="165.1"/>
@@
 <instance part="OSC1" gate="G$1" x="170.18" y="170.18"/>
 <instance part="SV1" gate="1" x="119.38" y="254" rot="R180"/>
-<instance part="SJ1" gate="1" x="256.54" y="223.52"/>
+<instance part="SJ1" gate="1" x="238.76" y="223.52" smashed="yes">
+<attribute name="NAME" x="241.3" y="220.98" size="1.778" layer="95"/>
+<attribute name="VALUE" x="236.22" y="219.71" size="1.778" layer="96"/>
+</instance>
 <instance part="IC6" gate="A1" x="426.72" y="226.06"/>
 <instance part="IC5" gate="G$1" x="111.76" y="228.6"/>
@@
 <instance part="R32" gate="G$1" x="73.66" y="187.96" rot="R90"/>
 <instance part="C4" gate="G$1" x="96.52" y="177.8"/>
+<instance part="C22" gate="G$1" x="203.2" y="91.44" rot="R90"/>
 </instances>
 <busses>
@@
 <segment>
 <wire x1="482.6" y1="187.96" x2="464.82" y2="187.96" width="0.1524" layer="91"/>
-<pinref part="C22" gate="G$1" pin="2"/>
-<wire x1="462.28" y1="193.04" x2="462.28" y2="187.96" width="0.1524" layer="91"/>
-<wire x1="462.28" y1="187.96" x2="464.82" y2="187.96" width="0.1524" layer="91"/>
 <wire x1="464.82" y1="187.96" x2="464.82" y2="185.42" width="0.1524" layer="91"/>
 <pinref part="SUPPLY3" gate="G$1" pin="DGND"/>
@@
 <junction x="419.1" y="187.96"/>
 <wire x1="426.72" y1="187.96" x2="439.42" y2="187.96" width="0.1524" layer="91"/>
-<junction x="462.28" y="187.96"/>
 <junction x="464.82" y="187.96"/>
 <junction x="426.72" y="187.96"/>
 <pinref part="C16" gate="G$1" pin="2"/>
-<wire x1="439.42" y1="187.96" x2="462.28" y2="187.96" width="0.1524" layer="91"/>
+<wire x1="439.42" y1="187.96" x2="464.82" y2="187.96" width="0.1524" layer="91"/>
 <wire x1="406.4" y1="218.44" x2="406.4" y2="213.36" width="0.1524" layer="91"/>
 <pinref part="IC6" gate="A1" pin="GND"/>
@@
 <segment>
 <pinref part="IC9" gate="G$1" pin="CPGND"/>
-<wire x1="190.5" y1="86.36" x2="195.58" y2="86.36" width="0.1524" layer="91"/>
+<wire x1="190.5" y1="86.36" x2="213.36" y2="86.36" width="0.1524" layer="91"/>
 <pinref part="IC9" gate="G$1" pin="AGND"/>
-<wire x1="190.5" y1="88.9" x2="195.58" y2="88.9" width="0.1524" layer="91"/>
-<wire x1="195.58" y1="86.36" x2="195.58" y2="88.9" width="0.1524" layer="91"/>
-<wire x1="195.58" y1="88.9" x2="213.36" y2="88.9" width="0.1524" layer="91"/>
+<wire x1="190.5" y1="88.9" x2="213.36" y2="88.9" width="0.1524" layer="91"/>
+<wire x1="213.36" y1="86.36" x2="213.36" y2="88.9" width="0.1524" layer="91"/>
 <wire x1="213.36" y1="88.9" x2="213.36" y2="91.44" width="0.1524" layer="91"/>
-<pinref part="R19" gate="G$1" pin="1"/>
 <wire x1="213.36" y1="91.44" x2="208.28" y2="91.44" width="0.1524" layer="91"/>
 <wire x1="213.36" y1="91.44" x2="223.52" y2="91.44" width="0.1524" layer="91"/>
 <label x="223.52" y="91.44" size="1.778" layer="95"/>
 <junction x="213.36" y="91.44"/>
-<junction x="195.58" y="88.9"/>
+<junction x="213.36" y="88.9"/>
+<pinref part="C22" gate="G$1" pin="2"/>
 </segment>
 <segment>
@@
 </segment>
 <segment>
-<wire x1="482.6" y1="205.74" x2="462.28" y2="205.74" width="0.1524" layer="91"/>
 <label x="482.6" y="205.74" size="1.778" layer="95" xref="yes"/>
-<pinref part="C22" gate="G$1" pin="1"/>
-<wire x1="462.28" y1="200.66" x2="462.28" y2="205.74" width="0.1524" layer="91"/>
-<junction x="462.28" y="205.74"/>
 <pinref part="IC7" gate="A1" pin="VO"/>
 <pinref part="C20" gate="G$1" pin="1"/>
@@
 <wire x1="419.1" y1="205.74" x2="426.72" y2="205.74" width="0.1524" layer="91"/>
 <wire x1="426.72" y1="205.74" x2="426.72" y2="200.66" width="0.1524" layer="91"/>
-<wire x1="426.72" y1="205.74" x2="462.28" y2="205.74" width="0.1524" layer="91"/>
+<wire x1="426.72" y1="205.74" x2="482.6" y2="205.74" width="0.1524" layer="91"/>
 <junction x="419.1" y="205.74"/>
 <junction x="426.72" y="205.74"/>
-</segment>
-<segment>
-<pinref part="L6" gate="G$1" pin="2"/>
-<wire x1="398.78" y1="132.08" x2="406.4" y2="132.08" width="0.1524" layer="91"/>
-<label x="406.4" y="132.08" size="1.778" layer="95" xref="yes"/>
 </segment>
 <segment>
@@
 <net name="N$1" class="0">
 <segment>
-<pinref part="R19" gate="G$1" pin="2"/>
 <pinref part="IC9" gate="G$1" pin="RFINB"/>
-<wire x1="198.12" y1="91.44" x2="190.5" y2="91.44" width="0.1524" layer="91"/>
+<wire x1="200.66" y1="91.44" x2="190.5" y2="91.44" width="0.1524" layer="91"/>
+<pinref part="C22" gate="G$1" pin="1"/>
 </segment>
 </net>
@@
 <segment>
 <pinref part="SJ1" gate="1" pin="2"/>
-<wire x1="261.62" y1="223.52" x2="266.7" y2="223.52" width="0.1524" layer="91"/>
-<label x="266.7" y="223.52" size="1.778" layer="95" xref="yes"/>
+<wire x1="243.84" y1="223.52" x2="256.54" y2="223.52" width="0.1524" layer="91"/>
+<label x="256.54" y="223.52" size="1.778" layer="95" xref="yes"/>
 </segment>
 </net>
@@
 <junction x="220.98" y="256.54"/>
 <pinref part="IC5" gate="G$1" pin="VCC"/>
-</segment>
-</net>
-<net name="CLK" class="0">
-<segment>
-<pinref part="IC9" gate="G$1" pin="CLK"/>
-<wire x1="157.48" y1="93.98" x2="139.7" y2="93.98" width="0.1524" layer="91"/>
-<label x="139.7" y="93.98" size="1.778" layer="95" rot="R180" xref="yes"/>
-</segment>
-<segment>
-<wire x1="419.1" y1="294.64" x2="403.86" y2="294.64" width="0.1524" layer="91"/>
-<label x="403.86" y="294.64" size="1.778" layer="95" rot="R180" xref="yes"/>
-<pinref part="IC4" gate="G$1" pin="CLK"/>
 </segment>
 </net>
@@
 <pinref part="TXFMR1" gate="G$1" pin="SEC_1"/>
 <wire x1="170.18" y1="345.44" x2="190.5" y2="345.44" width="0.1524" layer="91"/>
+<junction x="190.5" y="345.44"/>
 </segment>
 </net>
@@
 </segment>
 <segment>
-<wire x1="231.14" y1="223.52" x2="251.46" y2="223.52" width="0.1524" layer="91"/>
+<wire x1="231.14" y1="223.52" x2="233.68" y2="223.52" width="0.1524" layer="91"/>
+<pinref part="IC5" gate="G$1" pin="PB1_(MISO/DO/AIN1/OC0B/OC1A/PCINT1)"/>
+<label x="236.22" y="223.52" size="1.778" layer="95" rot="R180"/>
 <pinref part="SJ1" gate="1" pin="1"/>
-<pinref part="IC5" gate="G$1" pin="PB1_(MISO/DO/AIN1/OC0B/OC1A/PCINT1)"/>
 </segment>
 </net>
@@
 </segment>
 <segment>
-<wire x1="231.14" y1="226.06" x2="238.76" y2="226.06" width="0.1524" layer="91"/>
-<label x="238.76" y="226.06" size="1.778" layer="95" xref="yes"/>
+<wire x1="231.14" y1="226.06" x2="246.38" y2="226.06" width="0.1524" layer="91"/>
+<label x="246.38" y="226.06" size="1.778" layer="95" xref="yes"/>
 <pinref part="IC5" gate="G$1" pin="PB2_(SCK/USCK/SCL/ADC1/T0/INT0/PCINT2)"/>
+</segment>
+<segment>
+<wire x1="419.1" y1="294.64" x2="403.86" y2="294.64" width="0.1524" layer="91"/>
+<label x="403.86" y="294.64" size="1.778" layer="95" rot="R180" xref="yes"/>
+<pinref part="IC4" gate="G$1" pin="CLK"/>
+</segment>
+<segment>
+<pinref part="IC9" gate="G$1" pin="CLK"/>
+<wire x1="157.48" y1="93.98" x2="139.7" y2="93.98" width="0.1524" layer="91"/>
+<label x="139.7" y="93.98" size="1.778" layer="95" rot="R180" xref="yes"/>
 </segment>
 </net>
@@
 <wire x1="231.14" y1="220.98" x2="238.76" y2="220.98" width="0.1524" layer="91"/>
 <pinref part="IC5" gate="G$1" pin="PB0_(MOSI/DI/SDA/AIN0/OC0A/!OC1A!/AREF/PCINT0)"/>
+<label x="236.22" y="220.98" size="1.778" layer="95" rot="R180"/>
 </segment>
 </net>
@@
 </segment>
 </net>
+<net name="+5V_VCO" class="0">
+<segment>
+<pinref part="L6" gate="G$1" pin="2"/>
+<wire x1="398.78" y1="132.08" x2="406.4" y2="132.08" width="0.1524" layer="91"/>
+<label x="406.4" y="132.08" size="1.778" layer="95" xref="yes"/>
+</segment>
+</net>

Commit message: filter loop update
Parts:
- added C50: 100pF, resistor:C-EUC0603
- added C51: 100nF, resistor:C-EUC0603
- added L12: 100nH, resistor:R-EU_R0603
- added R19: 51R, rcl:R-EU_R0603
- C22: value 100pF -> 100nF; device resistor:C-EUC0603 -> rcl:C-EUC0805
- C43: value 6.8nF -> 27nF
- C44: value 22nF -> 10nF
- C45: value 10nF -> 1.2nF
- C46: value 15nF -> 100nF
- IC10: value TS971ILT -> MCP6H01T-E/LT; MPN TS971ILT -> MCP6H01T-E/LT; OC_FARNELL 9755730 -> 2920751
- R18: value 22R -> 18K
- R21: value 27k -> 560R
- R22: value 39k -> 560R
- R24: value 18K -> 10K
Connections:
- removed net +5V_VCO: L6.2
- removed net N$6: C43.2, IC10.OP, OSC2.CTRL, R24.2
- new net CLK: IC4.CLK, IC9.CLK
- new net N$39: L12.1, R24.2
- new net N$40: C51.2, OSC2.CTRL, R22.1
- net +3V3: now also L12.2
- net +9V: now also C22.1, L6.2
- net GND: now also C50.1, C51.1, R19.1
- net LOOP_IN: now also IC10.+, R21.2; no longer R21.1
- net N$1: now also R19.2; no longer C22.1
- net N$5: now also C46.2, C50.2
- net N$8: now also R21.1; no longer R21.2, R22.1
- net N$9: now also C43.2, IC10.OP; no longer C46.2, IC10.+
- net SCK: no longer IC4.CLK, IC9.CLK
Other:
- note removed: "Sallen-Key 500Hz LPF, Gain: 2.8"
- moved on the sheet: C22, C39, C40, C43, C46, L9, R21, R22, R24, R25, SJ1

Commit message: Layout
Parts:
- added C52: DNF, resistor:C-EUC0603
Connections:
- net LOOP_IN: now also C52.1
- net N$8: now also C52.2
Changed lines of the file:
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@@
 <part name="R22" library="rcl" deviceset="R-EU_" device="R0603" value="560R"/>
 <part name="C51" library="resistor" deviceset="C-EU" device="C0603" value="100nF"/>
+<part name="C52" library="resistor" deviceset="C-EU" device="C0603" value="DNF"/>
 </parts>
 <sheets>
@@
 <instance part="R22" gate="G$1" x="337.82" y="81.28" rot="R180"/>
 <instance part="C51" gate="G$1" x="345.44" y="68.58" rot="R180"/>
+<instance part="C52" gate="G$1" x="292.1" y="106.68" rot="R90"/>
 </instances>
 <busses>
@@
 <wire x1="287.02" y1="99.06" x2="287.02" y2="83.82" width="0.1524" layer="91"/>
 <junction x="287.02" y="83.82"/>
+<pinref part="C52" gate="G$1" pin="1"/>
+<wire x1="289.56" y1="106.68" x2="287.02" y2="106.68" width="0.1524" layer="91"/>
+<wire x1="287.02" y1="106.68" x2="287.02" y2="99.06" width="0.1524" layer="91"/>
+<junction x="287.02" y="99.06"/>
 </segment>
 </net>
@@
 <pinref part="R21" gate="G$1" pin="1"/>
 <pinref part="C43" gate="G$1" pin="1"/>
-<wire x1="299.72" y1="99.06" x2="320.04" y2="99.06" width="0.1524" layer="91"/>
+<wire x1="299.72" y1="99.06" x2="302.26" y2="99.06" width="0.1524" layer="91"/>
+<pinref part="C52" gate="G$1" pin="2"/>
+<wire x1="302.26" y1="99.06" x2="320.04" y2="99.06" width="0.1524" layer="91"/>
+<wire x1="297.18" y1="106.68" x2="302.26" y2="106.68" width="0.1524" layer="91"/>
+<wire x1="302.26" y1="106.68" x2="302.26" y2="99.06" width="0.1524" layer="91"/>
+<junction x="302.26" y="99.06"/>
 </segment>
 </net>
@@
 <pinref part="R22" gate="G$1" pin="2"/>
 <wire x1="332.74" y1="81.28" x2="330.2" y2="81.28" width="0.1524" layer="91"/>
-</segment>
-</net>
+<junction x="330.2" y="81.28"/>
+</segment>
+</net>
