File: 4001_4153_LO_V2.sch (EAGLE design)
At the start: 121 parts, among them IC1 74LVC2G17GV,125, IC10 MCP6H01T-E/LT, IC11 TL431AIDBZR, IC2 74LVC2G17GV,125, IC3 74LVC2G17GV,125, IC4 ADF4001BRUZ, IC5 ATTINY45V-10SU, IC6 7805DT, IC7 7809DT, IC8 LD1117AS33TR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

Commit message: Ref synth updates
Firmware working for ADF4001
Various board updates, ref input still needs works
Parts:
- added LSP2: LSP13, solpad:LSP13
Connections:
- net 20_MHZ renamed 10MHZ
- net 20_MHZ_4001 renamed 10_MHZ_4001
- removed net CLK: IC4.CLK, IC9.CLK
- new net +12V_OSC: C16.1, IC6.VI, LSP2.MP
- net +12V: no longer C16.1, IC6.VI
- net +3V3: now also IC3.VCC; no longer IC3.GND
- net GND: now also IC3.GND; no longer IC3.VCC
- net SCK: now also IC4.CLK, IC9.CLK
Changed lines of the file:
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@@
 <part name="C51" library="resistor" deviceset="C-EU" device="C0603" value="100nF"/>
 <part name="C52" library="resistor" deviceset="C-EU" device="C0603" value="DNF"/>
+<part name="LSP2" library="solpad" deviceset="LSP13" device=""/>
 </parts>
 <sheets>
@@
 <instance part="C51" gate="G$1" x="345.44" y="68.58" rot="R180"/>
 <instance part="C52" gate="G$1" x="292.1" y="106.68" rot="R90"/>
+<instance part="LSP2" gate="1" x="368.3" y="231.14"/>
 </instances>
 <busses>
@@
 </segment>
 <segment>
-<pinref part="IC3" gate="G$1" pin="VCC"/>
-<wire x1="320.04" y1="284.48" x2="312.42" y2="284.48" width="0.1524" layer="91"/>
-<wire x1="312.42" y1="284.48" x2="312.42" y2="274.32" width="0.1524" layer="91"/>
-<label x="312.42" y="274.32" size="1.778" layer="95" rot="R180"/>
-</segment>
-<segment>
 <pinref part="C6" gate="G$1" pin="2"/>
 <wire x1="205.74" y1="322.58" x2="205.74" y2="317.5" width="0.1524" layer="91"/>
@@
 <label x="132.08" y="251.46" size="1.778" layer="95"/>
 </segment>
+<segment>
+<pinref part="IC3" gate="G$1" pin="GND"/>
+<wire x1="345.44" y1="284.48" x2="347.98" y2="284.48" width="0.1524" layer="91"/>
+<wire x1="347.98" y1="284.48" x2="347.98" y2="274.32" width="0.1524" layer="91"/>
+<wire x1="345.44" y1="274.32" x2="347.98" y2="274.32" width="0.1524" layer="91"/>
+<junction x="347.98" y="274.32"/>
+<wire x1="347.98" y1="274.32" x2="350.52" y2="274.32" width="0.1524" layer="91"/>
+<label x="345.44" y="271.78" size="1.778" layer="95"/>
+</segment>
 </net>
 <net name="+12V" class="2">
 <segment>
+<pinref part="R30" gate="G$1" pin="1"/>
+<wire x1="58.42" y1="195.58" x2="48.26" y2="195.58" width="0.1524" layer="91"/>
+<label x="48.26" y="195.58" size="1.778" layer="95" rot="R180" xref="yes"/>
+</segment>
+<segment>
+<pinref part="C19" gate="G$1" pin="1"/>
 <pinref part="IC7" gate="A1" pin="VI"/>
-<pinref part="C19" gate="G$1" pin="1"/>
 <wire x1="391.16" y1="205.74" x2="381" y2="205.74" width="0.1524" layer="91"/>
 <wire x1="381" y1="205.74" x2="381" y2="203.2" width="0.1524" layer="91"/>
-<wire x1="381" y1="205.74" x2="378.46" y2="205.74" width="0.1524" layer="91"/>
-<label x="363.22" y="205.74" size="1.778" layer="95" rot="R180" xref="yes"/>
 <junction x="381" y="205.74"/>
-<wire x1="378.46" y1="205.74" x2="368.3" y2="205.74" width="0.1524" layer="91"/>
-<wire x1="368.3" y1="205.74" x2="363.22" y2="205.74" width="0.1524" layer="91"/>
-<wire x1="378.46" y1="205.74" x2="378.46" y2="226.06" width="0.1524" layer="91"/>
-<pinref part="C16" gate="G$1" pin="1"/>
-<pinref part="IC6" gate="A1" pin="VI"/>
-<wire x1="406.4" y1="226.06" x2="416.56" y2="226.06" width="0.1524" layer="91"/>
-<junction x="406.4" y="226.06"/>
-<wire x1="378.46" y1="226.06" x2="406.4" y2="226.06" width="0.1524" layer="91"/>
-<junction x="378.46" y="205.74"/>
+<wire x1="381" y1="205.74" x2="368.3" y2="205.74" width="0.1524" layer="91"/>
 <pinref part="LSP1" gate="1" pin="MP"/>
 <wire x1="368.3" y1="208.28" x2="368.3" y2="205.74" width="0.1524" layer="91"/>
 <junction x="368.3" y="205.74"/>
-</segment>
-<segment>
-<pinref part="R30" gate="G$1" pin="1"/>
-<wire x1="58.42" y1="195.58" x2="48.26" y2="195.58" width="0.1524" layer="91"/>
-<label x="48.26" y="195.58" size="1.778" layer="95" rot="R180" xref="yes"/>
+<wire x1="368.3" y1="205.74" x2="363.22" y2="205.74" width="0.1524" layer="91"/>
+<label x="363.22" y="205.74" size="1.778" layer="95" rot="R180" xref="yes"/>
 </segment>
 </net>
@@
 </segment>
 <segment>
-<pinref part="IC3" gate="G$1" pin="GND"/>
-<wire x1="345.44" y1="284.48" x2="350.52" y2="284.48" width="0.1524" layer="91"/>
 <label x="345.44" y="302.26" size="1.778" layer="95" rot="R180"/>
-<wire x1="350.52" y1="284.48" x2="350.52" y2="302.26" width="0.1524" layer="91"/>
-<wire x1="350.52" y1="302.26" x2="345.44" y2="302.26" width="0.1524" layer="91"/>
 <pinref part="R27" gate="G$1" pin="1"/>
-<wire x1="350.52" y1="302.26" x2="358.14" y2="302.26" width="0.1524" layer="91"/>
+<wire x1="345.44" y1="302.26" x2="347.98" y2="302.26" width="0.1524" layer="91"/>
+<wire x1="347.98" y1="302.26" x2="358.14" y2="302.26" width="0.1524" layer="91"/>
 <wire x1="358.14" y1="302.26" x2="368.3" y2="302.26" width="0.1524" layer="91"/>
 <wire x1="368.3" y1="302.26" x2="368.3" y2="299.72" width="0.1524" layer="91"/>
 <pinref part="R26" gate="G$1" pin="1"/>
 <wire x1="358.14" y1="299.72" x2="358.14" y2="302.26" width="0.1524" layer="91"/>
-<junction x="350.52" y="302.26"/>
 <junction x="358.14" y="302.26"/>
+<pinref part="IC3" gate="G$1" pin="VCC"/>
+<wire x1="320.04" y1="284.48" x2="314.96" y2="284.48" width="0.1524" layer="91"/>
+<wire x1="314.96" y1="284.48" x2="314.96" y2="294.64" width="0.1524" layer="91"/>
+<wire x1="314.96" y1="294.64" x2="347.98" y2="294.64" width="0.1524" layer="91"/>
+<wire x1="347.98" y1="294.64" x2="347.98" y2="302.26" width="0.1524" layer="91"/>
+<junction x="347.98" y="302.26"/>
 </segment>
 <segment>
@@
 </segment>
 </net>
-<net name="20_MHZ" class="0">
+<net name="10MHZ" class="0">
 <segment>
 <wire x1="193.04" y1="175.26" x2="185.42" y2="175.26" width="0.1524" layer="91"/>
@@
 </segment>
 </net>
-<net name="CLK" class="0">
-<segment>
-<pinref part="IC9" gate="G$1" pin="CLK"/>
-<wire x1="157.48" y1="93.98" x2="139.7" y2="93.98" width="0.1524" layer="91"/>
-<label x="139.7" y="93.98" size="1.778" layer="95" rot="R180" xref="yes"/>
-</segment>
-<segment>
-<wire x1="419.1" y1="294.64" x2="403.86" y2="294.64" width="0.1524" layer="91"/>
-<label x="403.86" y="294.64" size="1.778" layer="95" rot="R180" xref="yes"/>
-<pinref part="IC4" gate="G$1" pin="CLK"/>
-</segment>
-</net>
 <net name="N$19" class="0">
 <segment>
@@
 </segment>
 </net>
-<net name="20_MHZ_4001" class="0">
+<net name="10_MHZ_4001" class="0">
 <segment>
 <pinref part="C28" gate="G$1" pin="1"/>
@@
 <pinref part="TXFMR1" gate="G$1" pin="SEC_1"/>
 <wire x1="170.18" y1="345.44" x2="190.5" y2="345.44" width="0.1524" layer="91"/>
+<junction x="190.5" y="345.44"/>
 </segment>
 </net>
@@
 <label x="238.76" y="226.06" size="1.778" layer="95" xref="yes"/>
 <pinref part="IC5" gate="G$1" pin="PB2_(SCK/USCK/SCL/ADC1/T0/INT0/PCINT2)"/>
+</segment>
+<segment>
+<pinref part="IC9" gate="G$1" pin="CLK"/>
+<wire x1="157.48" y1="93.98" x2="139.7" y2="93.98" width="0.1524" layer="91"/>
+<label x="139.7" y="93.98" size="1.778" layer="95" rot="R180" xref="yes"/>
+</segment>
+<segment>
+<wire x1="419.1" y1="294.64" x2="403.86" y2="294.64" width="0.1524" layer="91"/>
+<label x="403.86" y="294.64" size="1.778" layer="95" rot="R180" xref="yes"/>
+<pinref part="IC4" gate="G$1" pin="CLK"/>
 </segment>
 </net>
@@
 </segment>
 </net>
+<net name="+12V_OSC" class="2">
+<segment>
+<pinref part="C16" gate="G$1" pin="1"/>
+<pinref part="IC6" gate="A1" pin="VI"/>
+<wire x1="406.4" y1="226.06" x2="416.56" y2="226.06" width="0.1524" layer="91"/>
+<junction x="406.4" y="226.06"/>
+<wire x1="363.22" y1="226.06" x2="368.3" y2="226.06" width="0.1524" layer="91"/>
+<pinref part="LSP2" gate="1" pin="MP"/>
+<wire x1="368.3" y1="226.06" x2="406.4" y2="226.06" width="0.1524" layer="91"/>
+<wire x1="368.3" y1="228.6" x2="368.3" y2="226.06" width="0.1524" layer="91"/>
+<junction x="368.3" y="226.06"/>
+<label x="363.22" y="226.06" size="1.778" layer="95" rot="R180" xref="yes"/>
+</segment>
+</net>
